File: RD56c_electronics/RD56c/ESP-12F.kicad_sch (KiCad schematic)
At the start: 42 parts, among them J301 Micro_SD_Card, SW301 boot, SW302 reset, U302 ESP32-S3, U304 USBLC6-2SC6, U7 W25Q128JVS, Y301 40 MHz

Commit message: added empty_sheet.kicad_wks to KiCAD folders
Parts:
- gave numbers to parts that had none: 6
- renumbered R13 to R303, U7 to U303
