File: RD56c_electronics/RD56c/LED_electronics2.kicad_sch (KiCad schematic)
At the start: 12 parts, among them IC1 STP24DP05BTR, IC2 STP24DP05BTR

Commit message: added empty_sheet.kicad_wks to KiCAD folders
Parts:
- renumbered C5 to C701, C4 to C702, C6 to C703, C7 to C704, R18 to R701, R23 to R702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
