File: RD56c_electronics/RD56c/LED_electronics3.kicad_sch (KiCad schematic)
At the start: 56 parts

Commit message: added empty_sheet.kicad_wks to KiCAD folders
Parts:
- renumbered C50 to C801, C50 to C802, C50 to C803, C50 to C804, C50 to C805, C50 to C806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
