File: RD56c_electronics/RD56c/LED_electronics4_sch.kicad_sch (KiCad schematic)
At the start: 56 parts

Commit message: added empty_sheet.kicad_wks to KiCAD folders
Parts:
- renumbered C50 to C901, C50 to C902, C50 to C903, C50 to C904, C50 to C905, C50 to C906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
