File: RD56c_electronics/RD56c/RP2040.kicad_sch (KiCad schematic)
At the start: 34 parts, among them SW401 reset, SW402 USB boot, U3 USBLC6-2SC6, U402 RP2040, U403 MH253, U404 W25Q128JVS

Commit message: added empty_sheet.kicad_wks to KiCAD folders
Parts:
- gave numbers to parts that had none: 24
- renumbered U3 to U401
